Commit message: rafsync

File: henrybot/henrybot_description/urdf/henry.urdf.xacro (robot description, xacro)
@@ -17,7 +17,17 @@
   <xacro:include filename="$(find henrybot_description)/urdf/table.urdf.xacro" />
   <xacro:table prefix="" />
+  <joint name="${prefix}table_to_mir" type="fixed">
+    <parent link="${prefix}base_footprint"/>
+    <child link="${prefix}table_mir"/>
+    <origin xyz="0.0 0.0 0.0" rpy="0.0 0.0 0.0"/>
+  </joint>
   <!-- UR5e -->
   <xacro:include filename="$(find ur_description)/urdf/inc/ur5e_macro.xacro"/>
-  <xacro:ur5e_robot prefix="" />
+  <xacro:ur5e_robot prefix="${prefix}ur5e_" />
+  <joint name="${prefix}ur_to_table" type="fixed">
+    <parent link="${prefix}table_mir"/>
+    <child link="${prefix}ur5e_base_link"/>
+    <origin xyz="0.325 0.0 0.85" rpy="0.0 0.0 0.0"/>
+  </joint>
   <!-- ROS-Industrial 'base' frame: base_link to UR 'Base' Coordinates transform -->
   <link name="${prefix}base"/>
@@ -35,11 +45,4 @@
   <xacro:include filename="$(find robotiq_2f_85_gripper_visualization)/urdf/robotiq_arg2f_85_model_macro.xacro" />
   <xacro:robotiq_arg2f_85 prefix=""/>
-  <link name="${prefix}tool0"/>
-    <joint name="${prefix}flange-tool0" type="fixed">
-      <!-- default toolframe: X+ left, Y+ up, Z+ front -->
-      <origin xyz="0 0 0" rpy="${pi/2.0} 0 ${pi/2.0}"/>
-      <parent link="${prefix}flange"/>
-      <child link="${prefix}tool0"/>
-    </joint>
   <joint name="${prefix}gripper_to_ur" type="fixed" >
     <parent link="${prefix}ur5e_tool0" />

File: henrybot/henrybot_description/urdf/table.urdf.xacro (robot description, xacro)
@@ -6,5 +6,5 @@
       <origin xyz="0.1 0 -0.1" rpy="1.57 0 1.57"/>
       <geometry>
-        <mesh filename="$(find henrybot_description)/meshes/table.stl"/>
+        <mesh filename="package://henrybot_description/meshes/table.stl"/>
       </geometry>
       <material name="LightGrey">
@@ -15,5 +15,5 @@
       <origin xyz="0.1 0 -0.1" rpy="1.57 0 1.57"/>
       <geometry>
-        <mesh filename="$(find henrybot_description)/meshes/table.stl"/>
+        <mesh filename="package://henrybot_description/meshes/table.stl"/>
       </geometry>
     </collision>

Commit message: rafsync

File: henrybot/henrybot_description/urdf/henry.urdf.xacro (robot description, xacro)
@@ -12,7 +12,7 @@
     <xacro:property name="prefix" value="${tf_prefix_}/" />
   </xacro:unless>
-  <xacro:mir_100 prefix="${prefix}"/>
+  <xacro:mir_250 prefix="${prefix}"/>
   <xacro:controller_plugin_gazebo robot_namespace=""/>
-  <!-- table -->
+  <!-- table from sdl-application.. need to fix it for our real table -->
   <xacro:include filename="$(find henrybot_description)/urdf/table.urdf.xacro" />
   <xacro:table prefix="" />
@@ -23,6 +23,29 @@
   </joint>
   <!-- UR5e -->
+  <xacro:macro name="ur5e_robot" params="
+   prefix
+   joint_limits_parameters_file:='$(find ur_description)/config/ur5e/joint_limits.yaml'
+   kinematics_parameters_file:='$(find ur_description)/config/ur5e/default_kinematics.yaml'
+   physical_parameters_file:='$(find ur_description)/config/ur5e/physical_parameters.yaml'
+   visual_parameters_file:='$(find ur_description)/config/ur5e/visual_parameters.yaml'
+   transmission_hw_interface:=hardware_interface/PositionJointInterface
+   safety_limits:=false
+   safety_pos_margin:=0.15
+   safety_k_position:=20"
+  >
   <xacro:include filename="$(find ur_description)/urdf/inc/ur5e_macro.xacro"/>
-  <xacro:ur5e_robot prefix="${prefix}ur5e_" />
+  <xacro:ur5e_robot
+    prefix="${prefix}ur5e_"
+    joint_limits_parameters_file="${joint_limits_parameters_file}"
+    kinematics_parameters_file="${kinematics_parameters_file}"
+    physical_parameters_file="${physical_parameters_file}"
+    visual_parameters_file="${visual_parameters_file}"
+    transmission_hw_interface="${transmission_hw_interface}"
+    safety_limits="${safety_limits}"
+    safety_pos_margin="${safety_pos_margin}"
+    safety_k_position="${safety_k_position}"
+  />
+  </xacro:macro>
+    <xacro:ur5e_robot prefix="" />
   <joint name="${prefix}ur_to_table" type="fixed">
     <parent link="${prefix}table_mir"/>

Commit message: sync

File: henrybot/henrybot_description/urdf/henry.urdf.xacro (robot description, xacro)
@@ -1,7 +1,4 @@
 <?xml version="1.0"?>
 <robot name="henry" xmlns:xacro="http://ros.org/wiki/xacro">
-  <!-- MiR100 base -->
-  <xacro:include filename="$(find mir_description)/urdf/include/mir_100_v1.urdf.xacro" />
-  <xacro:include filename="$(find mir_description)/urdf/include/common.gazebo.xacro" />
   <xacro:arg name="tf_prefix" default="" />
   <xacro:property name="tf_prefix_" value="$(arg tf_prefix)" />
@@ -12,7 +9,8 @@
     <xacro:property name="prefix" value="${tf_prefix_}/" />
   </xacro:unless>
-  <xacro:mir_250 prefix="${prefix}"/>
-  <xacro:controller_plugin_gazebo robot_namespace=""/>
-  <!-- table from sdl-application.. need to fix it for our real table -->
+  <!-- MiR250 base -->
+  <xacro:include filename="$(find mir_description)/urdf/include/mir_100_v1.urdf.xacro" />
+  <xacro:mir_100 prefix="${prefix}"/>
+  <!-- table -->
   <xacro:include filename="$(find henrybot_description)/urdf/table.urdf.xacro" />
   <xacro:table prefix="" />
@@ -23,29 +21,29 @@
   </joint>
   <!-- UR5e -->
-  <xacro:macro name="ur5e_robot" params="
-   prefix
-   joint_limits_parameters_file:='$(find ur_description)/config/ur5e/joint_limits.yaml'
-   kinematics_parameters_file:='$(find ur_description)/config/ur5e/default_kinematics.yaml'
-   physical_parameters_file:='$(find ur_description)/config/ur5e/physical_parameters.yaml'
-   visual_parameters_file:='$(find ur_description)/config/ur5e/visual_parameters.yaml'
-   transmission_hw_interface:=hardware_interface/PositionJointInterface
-   safety_limits:=false
-   safety_pos_margin:=0.15
-   safety_k_position:=20"
-  >
   <xacro:include filename="$(find ur_description)/urdf/inc/ur5e_macro.xacro"/>
-  <xacro:ur5e_robot
+   <!-- parameters -->
+   <xacro:arg name="joint_limit_params" default="$(find ur_description)/config/ur5e/joint_limits.yaml"/>
+   <xacro:arg name="kinematics_params" default="$(find ur_description)/config/ur5e/default_kinematics.yaml"/>
+   <xacro:arg name="physical_params" default="$(find ur_description)/config/ur5e/physical_parameters.yaml"/>
+   <xacro:arg name="visual_params" default="$(find ur_description)/config/ur5e/visual_parameters.yaml"/>
+   <!-- legal values:
+         - hardware_interface/PositionJointInterface
+         - hardware_interface/VelocityJointInterface
+         - hardware_interface/EffortJointInterface
+   -->
+   <xacro:arg name="transmission_hw_interface" default="hardware_interface/PositionJointInterface"/>
+   <xacro:arg name="safety_limits" default="false"/>
+   <xacro:arg name="safety_pos_margin" default="0.15"/>
+   <xacro:arg name="safety_k_position" default="20"/>
+   <xacro:ur5e_robot
     prefix="${prefix}ur5e_"
-    joint_limits_parameters_file="${joint_limits_parameters_file}"
-    kinematics_parameters_file="${kinematics_parameters_file}"
-    physical_parameters_file="${physical_parameters_file}"
-    visual_parameters_file="${visual_parameters_file}"
-    transmission_hw_interface="${transmission_hw_interface}"
-    safety_limits="${safety_limits}"
-    safety_pos_margin="${safety_pos_margin}"
-    safety_k_position="${safety_k_position}"
-  />
-  </xacro:macro>
-    <xacro:ur5e_robot prefix="" />
+     joint_limits_parameters_file="$(arg joint_limit_params)"
+     kinematics_parameters_file="$(arg kinematics_params)"
+     physical_parameters_file="$(arg physical_params)"
+     visual_parameters_file="$(arg visual_params)"
+     transmission_hw_interface="$(arg transmission_hw_interface)"
+     safety_limits="$(arg safety_limits)"
+     safety_pos_margin="$(arg safety_pos_margin)"
+     safety_k_position="$(arg safety_k_position)"/>
   <joint name="${prefix}ur_to_table" type="fixed">
     <parent link="${prefix}table_mir"/>

File: henrybot/henrybot_description/urdf/table.urdf.xacro (robot description, xacro)
@@ -9,5 +9,5 @@
       </geometry>
       <material name="LightGrey">
-        <color rgba="0.7 0.7 0.7 1.0"/>
+        <color rgba="0.0 0.0 0.8 0.8"/>
       </material>
     </visual>

Commit message: sync

File: henrybot/henrybot_description/urdf/henry.urdf.xacro (robot description, xacro)
@@ -11,62 +11,44 @@
   <!-- MiR250 base -->
   <xacro:include filename="$(find mir_description)/urdf/include/mir_100_v1.urdf.xacro" />
-  <xacro:mir_100 prefix="${prefix}"/>
+  <xacro:mir_100 prefix="${prefix}mir_"/>
   <!-- table -->
   <xacro:include filename="$(find henrybot_description)/urdf/table.urdf.xacro" />
-  <xacro:table prefix="" />
+  <xacro:table prefix="${prefix}"/>
+  <!-- UR5e -->
+  <xacro:include filename="$(find ur_description)/urdf/inc/ur5e_macro.xacro"/>
+  <xacro:ur5e_robot
+    prefix="${prefix}ur_"
+    joint_limits_parameters_file="$(find ur_description)/config/ur5e/joint_limits.yaml"
+    kinematics_parameters_file="$(find ur_description)/config/ur5e/default_kinematics.yaml"
+    physical_parameters_file="$(find ur_description)/config/ur5e/physical_parameters.yaml"
+    visual_parameters_file="$(find ur_description)/config/ur5e/visual_parameters.yaml"
+    transmission_hw_interface="hardware_interface/PositionJointInterface"
+    safety_limits="false"
+    safety_pos_margin="0.15"
+    safety_k_position="20"/>
+  <!-- Gripper -->
+  <xacro:include filename="$(find robotiq_2f_85_gripper_visualization)/urdf/robotiq_arg2f_85_model_macro.xacro" />
+  <xacro:robotiq_arg2f_85 prefix="${prefix}"/>
+  <!-- Montage Links -->
   <joint name="${prefix}table_to_mir" type="fixed">
-    <parent link="${prefix}base_footprint"/>
-    <child link="${prefix}table_mir"/>
+    <parent link="${prefix}mir_base_link"/>
+    <child link="${prefix}table"/>
     <origin xyz="0.0 0.0 0.0" rpy="0.0 0.0 0.0"/>
   </joint>
-  <!-- UR5e -->
-  <xacro:include filename="$(find ur_description)/urdf/inc/ur5e_macro.xacro"/>
-   <!-- parameters -->
-   <xacro:arg name="joint_limit_params" default="$(find ur_description)/config/ur5e/joint_limits.yaml"/>
-   <xacro:arg name="kinematics_params" default="$(find ur_description)/config/ur5e/default_kinematics.yaml"/>
-   <xacro:arg name="physical_params" default="$(find ur_description)/config/ur5e/physical_parameters.yaml"/>
-   <xacro:arg name="visual_params" default="$(find ur_description)/config/ur5e/visual_parameters.yaml"/>
-   <!-- legal values:
-         - hardware_interface/PositionJointInterface
-         - hardware_interface/VelocityJointInterface
-         - hardware_interface/EffortJointInterface
-   -->
-   <xacro:arg name="transmission_hw_interface" default="hardware_interface/PositionJointInterface"/>
-   <xacro:arg name="safety_limits" default="false"/>
-   <xacro:arg name="safety_pos_margin" default="0.15"/>
-   <xacro:arg name="safety_k_position" default="20"/>
-   <xacro:ur5e_robot
-    prefix="${prefix}ur5e_"
-     joint_limits_parameters_file="$(arg joint_limit_params)"
-     kinematics_parameters_file="$(arg kinematics_params)"
-     physical_parameters_file="$(arg physical_params)"
-     visual_parameters_file="$(arg visual_params)"
-     transmission_hw_interface="$(arg transmission_hw_interface)"
-     safety_limits="$(arg safety_limits)"
-     safety_pos_margin="$(arg safety_pos_margin)"
-     safety_k_position="$(arg safety_k_position)"/>
   <joint name="${prefix}ur_to_table" type="fixed">
-    <parent link="${prefix}table_mir"/>
-    <child link="${prefix}ur5e_base_link"/>
+    <parent link="${prefix}table"/>
+    <child link="${prefix}ur_base_link"/>
     <origin xyz="0.325 0.0 0.85" rpy="0.0 0.0 0.0"/>
   </joint>
-  <!-- ROS-Industrial 'base' frame: base_link to UR 'Base' Coordinates transform -->
-  <link name="${prefix}base"/>
-    <joint name="${prefix}base_link-base_fixed_joint" type="fixed">
-      <!-- Note the rotation over Z of pi radians: as base_link is REP-103
-           aligned (ie: has X+ forward, Y+ left and Z+ up), this is needed
-           to correctly align 'base' with the 'Base' coordinate system of
-           the UR controller.
-      -->
-      <origin xyz="0 0 0" rpy="0 0 ${pi}"/>
-      <parent link="${prefix}base_link"/>
-      <child link="${prefix}base"/>
-    </joint>
-  <!-- Gripper -->
-  <xacro:include filename="$(find robotiq_2f_85_gripper_visualization)/urdf/robotiq_arg2f_85_model_macro.xacro" />
-  <xacro:robotiq_arg2f_85 prefix=""/>
   <joint name="${prefix}gripper_to_ur" type="fixed" >
-    <parent link="${prefix}ur5e_tool0" />
+    <parent link="${prefix}ur_tool0" />
     <child link="${prefix}robotiq_arg2f_base_link" />
   </joint>
+  <!-- ROS-Industrial 'base' frame: base_link to UR 'Base' Coordinates transform -->
+  <!-- <link name="${prefix}ur_base"/>
+    <joint name="${prefix}ur_base_link-base_fixed_joint" type="fixed">
+      <origin xyz="0 0 0" rpy="0 0 ${pi}"/>
+      <parent link="${prefix}ur_base_link"/>
+      <child link="${prefix}ur_base"/>
+    </joint> -->
 </robot>

File: henrybot/henrybot_description/urdf/table.urdf.xacro (robot description, xacro)
@@ -2,5 +2,5 @@
 <robot xmlns:xacro="http://ros.org/wiki/xacro">
   <xacro:macro name="table" params="prefix">
-  <link name="${prefix}table_mir" >
+  <link name="${prefix}table" >
     <visual>
       <origin xyz="0.1 0 -0.1" rpy="1.57 0 1.57"/>

Commit message: casey

File: henrybot/henrybot_description/urdf/henry.urdf.xacro (robot description, xacro)
@@ -10,45 +10,43 @@
   </xacro:unless>
   <!-- MiR250 base -->
-  <xacro:include filename="$(find mir_description)/urdf/include/mir_100_v1.urdf.xacro" />
-  <xacro:mir_100 prefix="${prefix}mir_"/>
+  <xacro:include filename="$(find henrybot_description)/urdf/include/mir_100_v2.urdf.xacro" />
+  <xacro:mir_100 prefix="${prefix}mir/"/>
   <!-- table -->
-  <xacro:include filename="$(find henrybot_description)/urdf/table.urdf.xacro" />
+  <xacro:include filename="$(find henrybot_description)/urdf/include/table.urdf.xacro" />
   <xacro:table prefix="${prefix}"/>
   <!-- UR5e -->
-  <xacro:include filename="$(find ur_description)/urdf/inc/ur5e_macro.xacro"/>
-  <xacro:ur5e_robot
-    prefix="${prefix}ur_"
-    joint_limits_parameters_file="$(find ur_description)/config/ur5e/joint_limits.yaml"
-    kinematics_parameters_file="$(find ur_description)/config/ur5e/default_kinematics.yaml"
-    physical_parameters_file="$(find ur_description)/config/ur5e/physical_parameters.yaml"
-    visual_parameters_file="$(find ur_description)/config/ur5e/visual_parameters.yaml"
-    transmission_hw_interface="hardware_interface/PositionJointInterface"
-    safety_limits="false"
-    safety_pos_margin="0.15"
-    safety_k_position="20"/>
+  <xacro:include filename="$(find ur_description)/urdf/inc/ur_macro.xacro"/>
+   <!-- legal values:
+         - hardware_interface/PositionJointInterface
+         - hardware_interface/VelocityJointInterface
+         - hardware_interface/EffortJointInterface
+   -->
+   <xacro:ur_robot
+    prefix="${prefix}"
+     joint_limits_parameters_file="$(find ur_description)/config/ur5e/joint_limits.yaml"
+     kinematics_parameters_file="$(find ur_description)/config/ur5e/default_kinematics.yaml"
+     physical_parameters_file="$(find ur_description)/config/ur5e/physical_parameters.yaml"
+     visual_parameters_file="$(find ur_description)/config/ur5e/visual_parameters.yaml"
+     transmission_hw_interface="hardware_interface/PositionJointInterface"
+     safety_limits="false"
+     safety_pos_margin="0.15"
+     safety_k_position="20"/>
   <!-- Gripper -->
   <xacro:include filename="$(find robotiq_2f_85_gripper_visualization)/urdf/robotiq_arg2f_85_model_macro.xacro" />
   <xacro:robotiq_arg2f_85 prefix="${prefix}"/>
-  <!-- Montage Links -->
+  <!-- Connections -->
   <joint name="${prefix}table_to_mir" type="fixed">
-    <parent link="${prefix}mir_base_link"/>
+    <parent link="${prefix}mir/base_link"/>
     <child link="${prefix}table"/>
     <origin xyz="0.0 0.0 0.0" rpy="0.0 0.0 0.0"/>
   </joint>
-  <joint name="${prefix}ur_to_table" type="fixed">
-    <parent link="${prefix}table"/>
-    <child link="${prefix}ur_base_link"/>
-    <origin xyz="0.325 0.0 0.85" rpy="0.0 0.0 0.0"/>
+ <joint name="${prefix}ur_to_table" type="fixed">
+    <parent link="${prefix}mir/surface"/>
+    <child link="${prefix}base_link"/>
+    <origin xyz="0.3 0.0 0.6" rpy="0.0 0.0 0.0"/>
   </joint>
   <joint name="${prefix}gripper_to_ur" type="fixed" >
-    <parent link="${prefix}ur_tool0" />
+    <parent link="${prefix}tool0" />
     <child link="${prefix}robotiq_arg2f_base_link" />
   </joint>
-  <!-- ROS-Industrial 'base' frame: base_link to UR 'Base' Coordinates transform -->
-  <!-- <link name="${prefix}ur_base"/>
-    <joint name="${prefix}ur_base_link-base_fixed_joint" type="fixed">
-      <origin xyz="0 0 0" rpy="0 0 ${pi}"/>
-      <parent link="${prefix}ur_base_link"/>
-      <child link="${prefix}ur_base"/>
-    </joint> -->
 </robot>

Commit message: long sync

File: henrybot/henrybot_description/urdf/henry.urdf.xacro (robot description, xacro)
@@ -44,5 +44,5 @@
     <parent link="${prefix}mir/surface"/>
     <child link="${prefix}base_link"/>
-    <origin xyz="0.3 0.0 0.6" rpy="0.0 0.0 0.0"/>
+    <origin xyz="0.3 0.0 0.6" rpy="0.0 0.0 ${pi/2}"/>
   </joint>
   <joint name="${prefix}gripper_to_ur" type="fixed" >
